Commit message: Tensor Inertia is recomuputed to have zero rotation for axes of inertia, since Gazebo Ros does not support roation function; Scripts for comuting are in Octave scripts folder

File: youbot_common/youbot_description/urdf/youbot_arm/limits.urdf.xacro (robot description, xacro)
@@ -28,36 +28,31 @@
 	<xacro:macro name="link_1_inertia_tensor">
 		<origin xyz="${14.89/1000} ${2.13/1000} ${2.13/1000}"
-			rpy="${180.00*M_PI/180}  ${20.00*M_PI/180} ${0*M_PI/180}" />
-		<inertia ixx="0.0035070" ixy="0" ixz="0"
-			 iyy="0.0065526" iyz="0"
-			 izz="0.0063686" />
+			rpy="0 0 0" />
+<inertia ixx="0.003863 " ixy="-0.000979 " ixz="0.000000"  		 iyy="0.006196" iyz
+="0.000000" 		 izz="0.006369" />
 	</xacro:macro>
 	<xacro:macro name="link_2_inertia_tensor">
 		<origin xyz="${104.53/1000} ${1.7/1000} ${-2.97/1000}"
-			rpy="${-90.00*M_PI/180}  ${0.00*M_PI/180} ${-90*M_PI/180}" />
-		<inertia ixx="0.0044395" ixy="0" ixz="0"
-			 iyy="0.0008231" iyz="0"
-			 izz="0.004447" />
+			rpy="0 0 0" />
+<inertia ixx="0.000823 " ixy="0.000000 " ixz="-0.000000"  		 iyy="0.004447" iyz
+="0.000000" 		 izz="0.004439" />
 	</xacro:macro>
 	<xacro:macro name="link_3_inertia_tensor">
 		<origin xyz="${0.1/1000} ${96.7/1000} ${21.07/1000}"
-			rpy="${0.00*M_PI/180}  ${0.00*M_PI/180} ${90*M_PI/180}" />
-		<inertia ixx="0.0024588" ixy="0" ixz="0"
-			 iyy="0.0005354" iyz="0"
-			 izz="0.0025708" />
+		rpy="0 0 0" />
+<inertia ixx="0.002459 " ixy="0.000000 " ixz="0.000000"  		 iyy="0.002571" iyz=
+"-0.000000" 		 izz="0.000535" />
 	</xacro:macro>
 	<xacro:macro name="link_4_inertia_tensor">
 		<origin xyz="${0.11/1000} ${51.03/1000} ${-23.19/1000}"
-			rpy="${0.00*M_PI/180}  ${180.00*M_PI/180} ${40*M_PI/180}" />
-		<inertia ixx="0.0008688" ixy="0" ixz="0"
-			 iyy="0.0013669" iyz="0"
-			 izz="0.0008970" />
+		rpy="0 0 0"  />
+<inertia ixx="0.000869 " ixy="0.000000 " ixz="-0.000000"  		 iyy="0.001173" iyz
+="-0.000231" 		 izz="0.001091" />
 	</xacro:macro>
 	<xacro:macro name="link_5_inertia_tensor">
 		<origin xyz="${0/1000} ${1.15/1000} ${-16.83/1000}"
-			rpy="${0.00*M_PI/180}  ${90.00*M_PI/180} ${0*M_PI/180}" />
-		<inertia ixx="0.0003388" ixy="0" ixz="0"
-			 iyy="0.0002798" iyz="0"
-			 izz="0.0001191" />
+		rpy="0 0 0" />
+<inertia ixx="0.000280 " ixy="0.000000 " ixz="0.000000"  		 iyy="0.000339" iyz=
+"0.000000" 		 izz="0.000119" />
 	</xacro:macro>
 </robot>

Commit message: bugfix

File: youbot_common/youbot_description/urdf/youbot_arm/limits.urdf.xacro (robot description, xacro)
@@ -29,30 +29,25 @@
 		<origin xyz="${14.89/1000} ${2.13/1000} ${2.13/1000}"
 			rpy="0 0 0" />
-<inertia ixx="0.003863 " ixy="-0.000979 " ixz="0.000000"  		 iyy="0.006196" iyz
-="0.000000" 		 izz="0.006369" />
+		<inertia ixx="0.003863" ixy="-0.000979" ixz="0.000000" iyy="0.006196" iyz="0.000000" izz="0.006369" />
 	</xacro:macro>
 	<xacro:macro name="link_2_inertia_tensor">
 		<origin xyz="${104.53/1000} ${1.7/1000} ${-2.97/1000}"
 			rpy="0 0 0" />
-<inertia ixx="0.000823 " ixy="0.000000 " ixz="-0.000000"  		 iyy="0.004447" iyz
-="0.000000" 		 izz="0.004439" />
+		<inertia ixx="0.000823" ixy="0.000000" ixz="-0.000000" iyy="0.004447" iyz ="0.000000" izz="0.004439" />
 	</xacro:macro>
 	<xacro:macro name="link_3_inertia_tensor">
 		<origin xyz="${0.1/1000} ${96.7/1000} ${21.07/1000}"
-		rpy="0 0 0" />
-<inertia ixx="0.002459 " ixy="0.000000 " ixz="0.000000"  		 iyy="0.002571" iyz=
-"-0.000000" 		 izz="0.000535" />
+			rpy="0 0 0" />
+		<inertia ixx="0.002459" ixy="0.000000" ixz="0.000000" iyy="0.002571" iyz="-0.000000" izz="0.000535" />
 	</xacro:macro>
 	<xacro:macro name="link_4_inertia_tensor">
 		<origin xyz="${0.11/1000} ${51.03/1000} ${-23.19/1000}"
-		rpy="0 0 0"  />
-<inertia ixx="0.000869 " ixy="0.000000 " ixz="-0.000000"  		 iyy="0.001173" iyz
-="-0.000231" 		 izz="0.001091" />
+			rpy="0 0 0"  />
+		<inertia ixx="0.000869" ixy="0.000000" ixz="-0.000000" iyy="0.001173" iyz="-0.000231" izz="0.001091" />
 	</xacro:macro>
 	<xacro:macro name="link_5_inertia_tensor">
 		<origin xyz="${0/1000} ${1.15/1000} ${-16.83/1000}"
-		rpy="0 0 0" />
-<inertia ixx="0.000280 " ixy="0.000000 " ixz="0.000000"  		 iyy="0.000339" iyz=
-"0.000000" 		 izz="0.000119" />
+			rpy="0 0 0" />
+		<inertia ixx="0.000280" ixy="0.000000" ixz="0.000000" iyy="0.000339" iyz="0.000000" izz="0.000119" />
 	</xacro:macro>
 </robot>
