Commit message: started to implements effort control; model parameters update.

File: youbot_common/youbot_description/urdf/youbot_arm/arm.transmission.xacro (robot description, xacro)
@@ -4,4 +4,6 @@
        xmlns:interface="http://playerstage.sourceforge.net/gazebo/xmlschema/#interface"
        xmlns:xacro="http://ros.org/wiki/xacro">
+	<!-- reduction ratio doesn't affect the model-->
+	<!-- reduction ratio must not to be 0-->
 	<xacro:macro name="youbot_arm_transmission" params="name">
 		<transmission name="${name}_trans_1" type="pr2_mechanism_model/SimpleTransmission">

File: youbot_common/youbot_description/urdf/youbot_arm/arm.urdf.xacro (robot description, xacro)
@@ -44,11 +44,11 @@
 			<axis xyz="0 0 -1"/>
 			<!--<calibration rising="${arm_1_ref}" falling="${arm_1_ref}"/>-->
-			<dynamics damping="0.5" friction="0.5" />
+			<dynamics damping="1" friction="1" />
 			<!-- damping - N*s/m, N*s*m/rad -->
 			<!-- friction - N, N*m -->
-			<limit effort="1" velocity="${M_PI / 2.0}" lower="0" upper="${joint_1_limit}"/>
+			<limit effort="${9.5}" velocity="${M_PI / 2.0}" lower="0" upper="${joint_1_limit}"/>
 			<!--effort - N, N*m-->
 			<!--velocity - m/s, rad/s-->
-			<safety_controller k_position="20" k_velocity="100" soft_lower_limit="${threshold}" soft_upper_limit="${joint_1_limit_soft}" />
+			<safety_controller k_position="20" k_velocity="${9.5/M_PI / 2.0}" soft_lower_limit="${threshold}" soft_upper_limit="${joint_1_limit_soft}" />
 			<!--k_position N/m, N/rad-->
 			<!--k_velocity N*s/m, N*s*m/rad-->
@@ -83,7 +83,7 @@
 			<axis xyz="0 1 0"/>
 			<!--<calibration rising="${arm_2_ref}" falling="${arm_2_ref}"/>-->
-			<dynamics damping="0.5" friction="0.5" />
-			<limit effort="10" velocity="${M_PI / 2.0}" lower="0" upper="${joint_2_limit}"/>
-                        <safety_controller k_position="20" k_velocity="1.0" soft_lower_limit="${threshold}" soft_upper_limit="${joint_2_limit_soft}" />
+			<dynamics damping="1" friction="1" />
+			<limit effort="${9.5}" velocity="${M_PI / 2.0}" lower="0" upper="${joint_2_limit}"/>
+                        <safety_controller k_position="20" k_velocity="${2*9.5/M_PI}" soft_lower_limit="${threshold}" soft_upper_limit="${joint_2_limit_soft}" />
 		</joint>
 		<link name="${name}_link_2">
@@ -115,7 +115,7 @@
 			<axis xyz="0 1 0"/>
 			<!--<calibration rising="${arm_3_ref}" falling="${arm_3_ref}"/>-->
-			<dynamics damping="0.5" friction="0.5" />
-			<limit effort="1" velocity="${M_PI / 2.0}" lower="-${joint_3_limit}" upper="0"/>
-                        <safety_controller k_position="20" k_velocity="1.0" soft_lower_limit="-${joint_3_limit_soft}" soft_upper_limit="${threshold}" />
+			<dynamics damping="1" friction="1" />
+			<limit effort="${6}" velocity="${M_PI / 2.0}" lower="-${joint_3_limit}" upper="0"/>
+                        <safety_controller k_position="20" k_velocity="100" soft_lower_limit="-${joint_3_limit_soft}" soft_upper_limit="${threshold}" />
 		</joint>
 		<link name="${name}_link_3">
@@ -147,7 +147,7 @@
 			<axis xyz="0 1 0" />
 			<!--<calibration rising="${arm_4_ref}" falling="${arm_4_ref}"/>-->
-			<dynamics damping="0.5" friction="0.5" />
-			<limit effort="1" velocity="${M_PI / 2.0}" lower="0" upper="${joint_4_limit}"/>
-			<safety_controller k_position="20" k_velocity="1.0" soft_lower_limit="0" soft_upper_limit="${joint_4_limit_soft}" />
+			<dynamics damping="1" friction="1" />
+			<limit effort="${2}" velocity="${M_PI / 2.0}" lower="0" upper="${joint_4_limit}"/>
+			<safety_controller k_position="20" k_velocity="100" soft_lower_limit="0" soft_upper_limit="${joint_4_limit_soft}" />
 		</joint>
 		<link name="${name}_link_4">
@@ -179,7 +179,7 @@
 			<axis xyz="0 0 1" />
 			<!--<calibration rising="${arm_5_ref}" falling="${arm_5_ref}"/>-->
-			<dynamics damping="0.5" friction="0.5" />
+			<dynamics damping="1" friction="1" />
 			<limit effort="1" velocity="${M_PI / 2.0}" lower="0" upper="${joint_5_limit}" />
-                        <safety_controller k_position="20" k_velocity="1.0" soft_lower_limit="0" soft_upper_limit="${joint_5_limit_soft}" />
+                        <safety_controller k_position="20" k_velocity="100" soft_lower_limit="0" soft_upper_limit="${joint_5_limit_soft}" />
 		</joint>
 		<link name="${name}_link_5">

File: youbot_common/youbot_description/urdf/youbot_arm/limits.urdf.xacro (robot description, xacro)
@@ -26,4 +26,9 @@
         	<origin xyz="0 0 0" rpy="0 0 0"/> <!-- no data known -->
 	</xacro:macro>
+	<xacro:macro name="link_default_inertia_tensor">
+		<origin xyz="0 0 0"
+			rpy="0 0 0" />
+		<inertia ixx="0.1" ixy="0" ixz="0" iyy="0.1" iyz="0" izz="0.1" />
+	</xacro:macro>
 	<xacro:macro name="link_1_inertia_tensor">
 		<origin xyz="${14.89/1000} ${2.13/1000} ${2.13/1000}"
