Commit message: added correct masses for the arm

File: youbot_common/youbot_description/urdf/youbot_arm/arm.urdf.xacro (robot description, xacro)
@@ -18,5 +18,5 @@
 				<!--<origin xyz="0.023 0 0.006" rpy="0 0 0"/>-->
 				<origin xyz="0 0 0" rpy="0 0 0"/>
-				<mass value="5"/>
+				<mass value="${link_0_mass}"/>
 				<inertia ixx="0.01" ixy="0" ixz="0" iyy="0.01" iyz="0" izz="0.01" />
 			</inertial>
@@ -52,5 +52,5 @@
 				<!--<origin xyz="0 0 -0.003" rpy="0 0 0" />-->
 				<origin xyz="0 0 0" rpy="0 0 0" />
-				<mass value="1"/>
+				<mass value="${link_1_mass}"/>
 				<inertia ixx="0.01" ixy="0" ixz="0" iyy="0.01" iyz="0" izz="0.01" />
 			</inertial>
@@ -86,5 +86,5 @@
 				<!--<origin xyz="0.001 -0.041 0.074" rpy="0 0 0" />-->
 				<origin xyz="0 -0.032 0.078" rpy="0 0 0" />
-				<mass value="1"/>
+				<mass value="${link_2_mass}"/>
 				<inertia ixx="0.01" ixy="0" ixz="0" iyy="0.01" iyz="0" izz="0.01" />
 			</inertial>
@@ -120,5 +120,5 @@
 				<!--<origin xyz="0.000 0.025 0.067" rpy="0 0 0" />-->
 				<origin xyz="0.000 0.028 0.079" rpy="0 0 0" />
-				<mass value="1"/>
+				<mass value="${link_3_mass}"/>
 				<inertia ixx="0.01" ixy="0" ixz="0" iyy="0.01" iyz="0" izz="0.01" />
 			</inertial>
@@ -154,5 +154,5 @@
 				<!--<origin xyz="0 0 0.026" rpy="0 0 0"/>-->
 				<origin xyz="0 -0.010 0.029" rpy="0 0 0"/>
-				<mass value="1"/>
+				<mass value="${link_4_mass}"/>
 				<inertia ixx="0.01" ixy="0" ixz="0" iyy="0.01" iyz="0" izz="0.01" />
 			</inertial>
@@ -187,5 +187,5 @@
 			<inertial>
 				<origin xyz="0.03 0 -0.030" rpy="0 0 0" />
-				<mass value="1"/>
+				<mass value="${link_5_mass}"/>
 				<inertia ixx="0.01" ixy="0" ixz="0" iyy="0.01" iyz="0" izz="0.01" />
 			</inertial>

File: youbot_common/youbot_description/urdf/youbot_arm/limits.urdf.xacro (robot description, xacro)
@@ -4,5 +4,5 @@
 	<property name="M_PI" value="3.1415926535897931" />
         <property name="threshold" value="0.01" />
-	<!-- arm reference positions -->
+	<!-- arm limits positions (deg) -->
 	<property name="joint_1_limit" value="${M_PI * (169 + 169) / 180}" />
 	<property name="joint_2_limit" value="${M_PI * (90 + 65) / 180}" />
@@ -15,3 +15,11 @@
 	<property name="joint_4_limit_soft" value="${M_PI * (102.5 + 102.5) / 180 - threshold}" />
 	<property name="joint_5_limit_soft" value="${M_PI * (167.5 + 167.5) / 180 - threshold}" />
+	<!-- dynamic properties : mass (kg)  -->
+	<property name="link_0_mass" value="0.845" />
+	<property name="link_1_mass" value="2.412" />
+	<property name="link_2_mass" value="1.155" />
+	<property name="link_3_mass" value="0.934" />
+	<property name="link_4_mass" value="0.877" />
+	<property name="link_5_mass" value="0.251" />
+	<!-- TODO: add inertia tensor-->
 </robot>

Commit message: started to tune the model, fixint time_from_start problem

File: youbot_common/youbot_description/urdf/youbot_arm/arm.urdf.xacro (robot description, xacro)
@@ -44,7 +44,14 @@
 			<axis xyz="0 0 -1"/>
 			<!--<calibration rising="${arm_1_ref}" falling="${arm_1_ref}"/>-->
-			<dynamics damping="1.0" friction="1.0" />
-			<limit effort="10" velocity="${M_PI / 2.0}" lower="0" upper="${joint_1_limit}"/>
-			<safety_controller k_position="20" k_velocity="25" soft_lower_limit="${threshold}" soft_upper_limit="${joint_1_limit_soft}" />
+			<dynamics damping="0.5" friction="0.5" />
+			<!-- damping - N*s/m, N*s*m/rad -->
+			<!-- friction - N, N*m -->
+			<limit effort="1" velocity="${M_PI / 2.0}" lower="0" upper="${joint_1_limit}"/>
+			<!--effort - N, N*m-->
+			<!--velocity - m/s, rad/s-->
+			<safety_controller k_position="20" k_velocity="100" soft_lower_limit="${threshold}" soft_upper_limit="${joint_1_limit_soft}" />
+			<!--k_position N/m, N/rad-->
+			<!--k_velocity N*s/m, N*s*m/rad-->
+			<!--for details: http://www.ros.org/wiki/pr2_controller_manager/safety_limits-->
 		</joint>
 		<link name="${name}_link_1">
@@ -78,7 +85,7 @@
 			<axis xyz="0 1 0"/>
 			<!--<calibration rising="${arm_2_ref}" falling="${arm_2_ref}"/>-->
-			<dynamics damping="1.0" friction="1.0" />
-			<limit effort="10" velocity="${M_PI / 2.0}" lower="0" upper="${joint_2_limit}"/>
-                        <safety_controller k_position="20" k_velocity="25" soft_lower_limit="${threshold}" soft_upper_limit="${joint_2_limit_soft}" />
+			<dynamics damping="0.5" friction="0.5" />
+			<limit effort="1" velocity="${M_PI / 2.0}" lower="0" upper="${joint_2_limit}"/>
+                        <safety_controller k_position="20" k_velocity="1.0" soft_lower_limit="${threshold}" soft_upper_limit="${joint_2_limit_soft}" />
 		</joint>
 		<link name="${name}_link_2">
@@ -112,7 +119,7 @@
 			<axis xyz="0 1 0"/>
 			<!--<calibration rising="${arm_3_ref}" falling="${arm_3_ref}"/>-->
-			<dynamics damping="1.0" friction="1.0" />
-			<limit effort="10" velocity="${M_PI / 2.0}" lower="-${joint_3_limit}" upper="0"/>
-                        <safety_controller k_position="20" k_velocity="25" soft_lower_limit="-${joint_3_limit_soft}" soft_upper_limit="${threshold}" />
+			<dynamics damping="0.5" friction="0.5" />
+			<limit effort="1" velocity="${M_PI / 2.0}" lower="-${joint_3_limit}" upper="0"/>
+                        <safety_controller k_position="20" k_velocity="1.0" soft_lower_limit="-${joint_3_limit_soft}" soft_upper_limit="${threshold}" />
 		</joint>
 		<link name="${name}_link_3">
@@ -146,7 +153,7 @@
 			<axis xyz="0 1 0" />
 			<!--<calibration rising="${arm_4_ref}" falling="${arm_4_ref}"/>-->
-			<dynamics damping="1.0" friction="1.0" />
-			<limit effort="10" velocity="${M_PI / 2.0}" lower="0" upper="${joint_4_limit}"/>
-			<safety_controller k_position="20" k_velocity="25" soft_lower_limit="0" soft_upper_limit="${joint_4_limit_soft}" />
+			<dynamics damping="0.5" friction="0.5" />
+			<limit effort="1" velocity="${M_PI / 2.0}" lower="0" upper="${joint_4_limit}"/>
+			<safety_controller k_position="20" k_velocity="1.0" soft_lower_limit="0" soft_upper_limit="${joint_4_limit_soft}" />
 		</joint>
 		<link name="${name}_link_4">
@@ -180,7 +187,7 @@
 			<axis xyz="0 0 1" />
 			<!--<calibration rising="${arm_5_ref}" falling="${arm_5_ref}"/>-->
-			<dynamics damping="1.0" friction="1.0" />
-			<limit effort="10" velocity="${M_PI / 2.0}" lower="0" upper="${joint_5_limit}" />
-                        <safety_controller k_position="20" k_velocity="25" soft_lower_limit="0" soft_upper_limit="${joint_5_limit_soft}" />
+			<dynamics damping="0.5" friction="0.5" />
+			<limit effort="1" velocity="${M_PI / 2.0}" lower="0" upper="${joint_5_limit}" />
+                        <safety_controller k_position="20" k_velocity="1.0" soft_lower_limit="0" soft_upper_limit="${joint_5_limit_soft}" />
 		</joint>
 		<link name="${name}_link_5">

Commit message: working on arm velocitity control for gazebo simulation

File: youbot_common/youbot_description/urdf/youbot_arm/arm.urdf.xacro (robot description, xacro)
@@ -86,5 +86,5 @@
 			<!--<calibration rising="${arm_2_ref}" falling="${arm_2_ref}"/>-->
 			<dynamics damping="0.5" friction="0.5" />
-			<limit effort="1" velocity="${M_PI / 2.0}" lower="0" upper="${joint_2_limit}"/>
+			<limit effort="10" velocity="${M_PI / 2.0}" lower="0" upper="${joint_2_limit}"/>
                         <safety_controller k_position="20" k_velocity="1.0" soft_lower_limit="${threshold}" soft_upper_limit="${joint_2_limit_soft}" />
 		</joint>

Commit message: added xacro for inertia tesor

File: youbot_common/youbot_description/urdf/youbot_arm/arm.urdf.xacro (robot description, xacro)
@@ -58,7 +58,8 @@
 			<inertial>
 				<!--<origin xyz="0 0 -0.003" rpy="0 0 0" />-->
-				<origin xyz="0 0 0" rpy="0 0 0" />
+				<!--<origin xyz="0 0 0" rpy="0 0 0" /> -->
 				<mass value="${link_1_mass}"/>
-				<inertia ixx="0.01" ixy="0" ixz="0" iyy="0.01" iyz="0" izz="0.01" />
+			        <!--<inertia ixx="0.01" ixy="0" ixz="0" iyy="0.01" iyz="0" izz="0.01" /> -->
+				<xacro: link_1_inertia_tensor />
 			</inertial>
 			<visual>

File: youbot_common/youbot_description/urdf/youbot_arm/limits.urdf.xacro (robot description, xacro)
@@ -15,5 +15,5 @@
 	<property name="joint_4_limit_soft" value="${M_PI * (102.5 + 102.5) / 180 - threshold}" />
 	<property name="joint_5_limit_soft" value="${M_PI * (167.5 + 167.5) / 180 - threshold}" />
-	<!-- dynamic properties : mass (kg)  -->
+	<!-- dynamic properties : mass (kg) Alu data sheet -->
 	<property name="link_0_mass" value="0.845" />
 	<property name="link_1_mass" value="2.412" />
@@ -23,3 +23,158 @@
 	<property name="link_5_mass" value="0.251" />
 	<!-- TODO: add inertia tensor-->
+	<xacro:macro name="default_origin">
+        	<origin xyz="0 0 0" rpy="0 0 0"/> <!-- no data known -->
+	</xacro:macro>
+	<xacro:macro name="link_1_inertia_tensor">
+		<origin xyz="${14.89/1000} ${2.13/1000} ${2.13/1000}"
+			rpy="${180.00*M_PI/180}  ${20.00*M_PI/180} ${0*M_PI/180}" />
+		<inertia ixx="0.0035070" ixy="0" ixz="0"
+				iyy="0.0065526" iyz="0"
+				        izz="0.0063686" />
+	</xacro:macro>
 </robot>
+<!--
+<?xml version="1.0" encoding="UTF-8"?>
+<DynDat xmlns:xsi="http://www.w3.org/2001/XMLSchema-instance" xsi:noNamespaceSchemaLocation="AxisData.xsd">
+  <Axis Number="1">
+    <Geometry>
+      <Mass m="2.412"/>
+      <CM-Frame x="14.89" y="2.13" z="31.05" a="180.00" b="20.00" c="0.00"/>
+      <Inertia xx="0.0035070" yy="0.0065526" zz="0.0063686"/>
+    </Geometry>
+    <Gear>
+      <DynamicLimits Mg="9.5" TrqTol="150" Mg_EM="40.0" Jerk="105263.203125"/>
+      <TorqueCharLine>
+        <x-Axis x1="0.00" x2="3.531" x3="0.00" x4="0.00" x5="0.00" x6="0.00" x7="0.00"/>
+        <y-Axis y1="9.500" y2="9.50" y3="0.00" y4="0.00" y5="0.00" y6="0.00" y7="0.00"/>
+      </TorqueCharLine>
+      <Friction Rh="0.00" Rv="0.00" Rz="1.00" Ad="1.00"/>
+    </Gear>
+    <Motor>
+      <Inertia Ja="0.3285"/>
+      <DynamicLimits Ma="0.084" S="1.000000" Ma_EM="40.0" TrqBrkMax="40.0" TrqBrkHold="40.000000" MaxEKin="7813.399902"/>
+      <TorqueCharLine>
+        <x-Axis x1="0.000" x2="550.8733" x3="0.00" x4="0.00" x5="0.00" x6="0.00" x7="0.00"/>
+        <y-Axis y1="0.084" y2="0.084000" y3="0.00" y4="0.00" y5="0.00" y6="0.00" y7="0.00"/>
+      </TorqueCharLine>
+    </Motor>
+    <AdditionalLoad>
+      <Mass m="0.00"/>
+      <CM-Frame x="0.00" y="0.00" z="0.00" a="0.00" b="0.00" c="0.00"/>
+      <Inertia xx="0.00" yy="0.00" zz="0.00"/>
+    </AdditionalLoad>
+  </Axis>
+  <Axis Number="2">
+    <Geometry>
+      <Mass m="1.155"/>
+      <CM-Frame x="104.53" y="1.70" z="-2.97" a="-90.00" b="0.00" c="-90.00"/>
+      <Inertia xx="0.0044395" yy="0.0008231" zz="0.004447"/>
+    </Geometry>
+    <Gear>
+      <DynamicLimits Mg="9.5" TrqTol="150" Mg_EM="40.0" Jerk="105263.203125"/>
+      <TorqueCharLine>
+        <x-Axis x1="0.0" x2="3.531" x3="0.00" x4="0.00" x5="0.00" x6="0.00" x7="0.00"/>
+        <y-Axis y1="9.50" y2="9.50" y3="0.00" y4="0.00" y5="0.00" y6="0.00" y7="0.00"/>
+      </TorqueCharLine>
+      <Friction Rh="0.00" Rv="0.00" Rz="1.00" Ad="1.00"/>
+    </Gear>
+    <Motor>
+       <Inertia Ja="0.3285"/>
+       <DynamicLimits Ma="0.084" S="1.000000" Ma_EM="40.0" TrqBrkMax="40.0" TrqBrkHold="40.000000" MaxEKin="7813.399902"/>
+       <TorqueCharLine>
+         <x-Axis x1="0.000" x2="550.88" x3="0.00" x4="0.00" x5="0.00" x6="0.00" x7="0.00"/>
+         <y-Axis y1="0.084" y2="0.0840" y3="0.00" y4="0.00" y5="0.00" y6="0.00" y7="0.00"/>
+       </TorqueCharLine>
+    </Motor>
+    <AdditionalLoad>
+      <Mass m="0.00"/>
+      <CM-Frame x="0.00" y="0.00" z="0.00" a="0.00" b="0.00" c="0.00"/>
+      <Inertia xx="0.00" yy="0.00" zz="0.00"/>
+    </AdditionalLoad>
+  </Axis>
+  <Axis Number="3">
+    <Geometry>
+      <Mass m="0.934"/>
+      <CM-Frame x="0.1" y="96.7" z="21.07" a="0.00" b="0.00" c="90.00"/>
+      <Inertia xx="0.0024588" yy="0.0005354" zz="0.0025708"/>
+    </Geometry>
+    <Gear>
+      <DynamicLimits Mg="6.0" TrqTol="150" Mg_EM="30.0" Jerk="105263.203125"/>
+      <TorqueCharLine>
+        <x-Axis x1="0.00" x2="5.73" x3="0.00" x4="0.00" x5="0.00" x6="0.00" x7="0.00"/>
+        <y-Axis y1="6.00" y2="6.00" y3="0.00" y4="0.00" y5="0.00" y6="0.00" y7="0.00"/>
+      </TorqueCharLine>
+      <Friction Rh="0.00" Rv="0.00" Rz="1.00" Ad="1.00"/>
+    </Gear>
+    <Motor>
+       <Inertia Ja="0.3285"/>
+       <DynamicLimits Ma="0.084" S="1.000000" Ma_EM="30.0" TrqBrkMax="30.0" TrqBrkHold="30.000000" MaxEKin="7813.399902"/>
+       <TorqueCharLine>
+         <x-Axis x1="0.000" x2="572.96" x3="0.00" x4="0.00" x5="0.00" x6="0.00" x7="0.00"/>
+         <y-Axis y1="0.084" y2="0.0840" y3="0.00" y4="0.00" y5="0.00" y6="0.00" y7="0.00"/>
+       </TorqueCharLine>
+    </Motor>
+    <AdditionalLoad>
+      <Mass m="0.00"/>
+      <CM-Frame x="0.00" y="0.00" z="0.00" a="0.00" b="0.00" c="0.00"/>
+      <Inertia xx="0.00" yy="0.00" zz="0.00"/>
+    </AdditionalLoad>
+  </Axis>
+  <Axis Number="4">
+    <Geometry>
+      <Mass m="0.877"/>
+      <CM-Frame x="0.11" y="51.03" z="-23.19" a="0.00" b="180.00" c="40.00"/>
+      <Inertia xx="0.0008688" yy="0.0013669" zz="0.0008970"/>
+    </Geometry>
+    <Gear>
+      <DynamicLimits Mg="2.0" TrqTol="150" Mg_EM="40.0" Jerk="105263.203125"/>
+      <TorqueCharLine>
+        <x-Axis x1="0.00" x2="11.29" x3="0.00" x4="0.00" x5="0.00" x6="0.00" x7="0.00"/>
+        <y-Axis y1="2.00" y2="2.000" y3="0.00" y4="0.00" y5="0.00" y6="0.00" y7="0.00"/>
+      </TorqueCharLine>
+      <Friction Rh="0.00" Rv="0.00" Rz="1.00" Ad="1.00"/>
+    </Gear>
+    <Motor>
+      <Inertia Ja="0.0466"/>
+      <DynamicLimits Ma="0.0588" S="1.00" Ma_EM="10.0" TrqBrkMax="10.0" TrqBrkHold="10.0" MaxEKin="636.200012"/>
+      <TorqueCharLine>
+        <x-Axis x1="0.0000" x2="802.14" x3="0.00" x4="0.00" x5="0.00" x6="0.00" x7="0.00"/>
+        <y-Axis y1="0.0466" y2="0.0466" y3="0.00" y4="0.00" y5="0.00" y6="0.00" y7="0.00"/>
+      </TorqueCharLine>
+    </Motor>
+    <AdditionalLoad>
+      <Mass m="0.00"/>
+      <CM-Frame x="0.00" y="0.00" z="0.00" a="0.00" b="0.00" c="0.00"/>
+      <Inertia xx="0.00" yy="0.00" zz="0.00"/>
+    </AdditionalLoad>
+  </Axis>
+  <Axis Number="5">
+    <Geometry>
+      <Mass m="0.251"/>
+      <CM-Frame x="0.00" y="1.15" z="-16.83" a="0.00" b="90.00" c="0.00"/>
+      <Inertia xx="0.0003388" yy="0.0002798" zz="0.0001191"/>
+    </Geometry>
+    <Gear>
+      <DynamicLimits Mg="1.0" TrqTol="150" Mg_EM="5.000" Jerk="30263.199219"/>
+      <TorqueCharLine>
+        <x-Axis x1="0.00" x2="11.57" x3="0.00" x4="0.00" x5="0.00" x6="0.00" x7="0.00"/>
+        <y-Axis y1="5.00" y2="5.000" y3="0.00" y4="0.00" y5="0.00" y6="0.00" y7="0.00"/>
+      </TorqueCharLine>
+      <Friction Rh="0.00" Rv="0.00" Rz="1.00" Ad="1.00"/>
+    </Gear>
+    <Motor>
+      <Inertia Ja="0.0176"/>
+      <DynamicLimits Ma="0.0233" S="1.00" Ma_EM="5.00" TrqBrkMax="5.00" TrqBrkHold="5.00" MaxEKin="963.400024"/>
+      <TorqueCharLine>
+        <x-Axis x1="0.0000" x2="821.24" x3="0.00" x4="0.00" x5="0.00" x6="0.00" x7="0.00"/>
+        <y-Axis y1="0.0233" y2="0.0233" y3="0.00" y4="0.00" y5="0.00" y6="0.00" y7="0.00"/>
+      </TorqueCharLine>
+    </Motor>
+    <AdditionalLoad>
+      <Mass m="0.400"/>
+      <CM-Frame x="0.00" y="0.00" z="28.9" a="180.00" b="0.00" c="90.00"/>
+      <Inertia xx="0.0003098" yy="0.0004771" zz="0.0002781"/>
+    </AdditionalLoad>
+  </Axis>
+ </DynDat>
+-->
