Commit message: fixing gazebo model, safety limits, correct axis directions and limits

File: youbot_common/youbot_description/urdf/youbot_arm/arm.urdf.xacro (robot description, xacro)
@@ -109,13 +109,21 @@
 		</link>
 		<!-- joint between arm_2_link and arm_3_link -->
+		<!--<joint name="${name}_joint_3" type="revolute">
+			<origin xyz="0.000 0.000 0.155" rpy="0 ${146 * M_PI / 180} 0"/>
+			<parent link="${name}_link_2"/>
+			<child link="${name}_link_3"/>
+			<axis xyz="0 1 0"/>
+			<dynamics damping="1" friction="1" />
+			<limit effort="${6}" velocity="${M_PI / 2.0}" lower="-${joint_3_limit}" upper="0"/>
+                        <safety_controller k_position="20" k_velocity="50" soft_lower_limit="-${joint_3_limit_soft}" soft_upper_limit="${threshold}" />
+		</joint>-->
 		<joint name="${name}_joint_3" type="revolute">
 			<origin xyz="0.000 0.000 0.155" rpy="0 ${146 * M_PI / 180} 0"/>
 			<parent link="${name}_link_2"/>
 			<child link="${name}_link_3"/>
-			<axis xyz="0 1 0"/>
-			<!--<calibration rising="${arm_3_ref}" falling="${arm_3_ref}"/>-->
-			<dynamics damping="1" friction="1" />
-			<limit effort="${6}" velocity="${M_PI / 2.0}" lower="-${joint_3_limit}" upper="0"/>
-                        <safety_controller k_position="20" k_velocity="100" soft_lower_limit="-${joint_3_limit_soft}" soft_upper_limit="${threshold}" />
+			<axis xyz="0 -1 0"/>
+			<dynamics damping="1" friction="1" />
+			<limit effort="${6}" velocity="${M_PI / 2.0}" lower="0" upper="${joint_3_limit}"/>
+                        <safety_controller k_position="20" k_velocity="50" soft_lower_limit="${threshold}" soft_upper_limit="${joint_3_limit_soft}" />
 		</joint>
 		<link name="${name}_link_3">
@@ -177,5 +185,5 @@
 			<parent link="${name}_link_4"/>
 			<child link="${name}_link_5"/>
-			<axis xyz="0 0 1" />
+			<axis xyz="0 0 -1" />
 			<!--<calibration rising="${arm_5_ref}" falling="${arm_5_ref}"/>-->
 			<dynamics damping="1" friction="1" />

File: youbot_common/youbot_description/urdf/youbot_arm/limits.urdf.xacro (robot description, xacro)
@@ -16,16 +16,16 @@
 	<property name="joint_5_limit_soft" value="${M_PI * (167.5 + 167.5) / 180 - threshold}" />
 	<!-- dynamic properties : mass (kg) Alu data sheet -->
-	<!--<property name="link_0_mass" value="0.845" />
+	<property name="link_0_mass" value="0.845" />
 	<property name="link_1_mass" value="2.412" />
 	<property name="link_2_mass" value="1.155" />
 	<property name="link_3_mass" value="0.934" />
 	<property name="link_4_mass" value="0.877" />
-	<property name="link_5_mass" value="0.251" />-->
-	<property name="link_0_mass" value="0.845" />
+	<property name="link_5_mass" value="0.251" />
+	<!--<property name="link_0_mass" value="0.845" />
 	<property name="link_1_mass" value="0.1" />
 	<property name="link_2_mass" value="0.1" />
 	<property name="link_3_mass" value="0.1" />
 	<property name="link_4_mass" value="0.1" />
-	<property name="link_5_mass" value="0.1" />
+	<property name="link_5_mass" value="0.1" />-->
 	<!-- TODO: add inertia tensor-->
 	<xacro:macro name="default_origin">

Commit message: added interaction controller for the youbot arm

File: youbot_common/youbot_description/urdf/youbot_arm/arm.urdf.xacro (robot description, xacro)
@@ -44,9 +44,4 @@
 			<axis xyz="0 0 -1"/>
 			<!--<calibration rising="${arm_1_ref}" falling="${arm_1_ref}"/>-->
-<<<<<<< HEAD
-			<dynamics damping="1.0" friction="1.0" />
-			<limit effort="10" velocity="${M_PI / 2.0}" lower="0" upper="${joint_1_limit}"/>
-			<safety_controller k_position="20" k_velocity="25" soft_lower_limit="${threshold}" soft_upper_limit="${joint_1_limit_soft}" />
-=======
 			<dynamics damping="1" friction="1" />
 			<!-- damping - N*s/m, N*s*m/rad -->
@@ -59,17 +54,9 @@
 			<!--k_velocity N*s/m, N*s*m/rad-->
 			<!--for details: http://www.ros.org/wiki/pr2_controller_manager/safety_limits-->
->>>>>>> working
 		</joint>
 		<link name="${name}_link_1">
 			<inertial>
-<<<<<<< HEAD
-				<!--<origin xyz="0 0 -0.003" rpy="0 0 0" />-->
-				<origin xyz="0 0 0" rpy="0 0 0" />
-				<mass value="${link_1_mass}"/>
-				<inertia ixx="0.01" ixy="0" ixz="0" iyy="0.01" iyz="0" izz="0.01" />
-=======
 				<mass value="${link_1_mass}"/>
 				<xacro:link_1_inertia_tensor />
->>>>>>> working
 			</inertial>
 			<visual>
@@ -96,13 +83,7 @@
 			<axis xyz="0 1 0"/>
 			<!--<calibration rising="${arm_2_ref}" falling="${arm_2_ref}"/>-->
-<<<<<<< HEAD
-			<dynamics damping="1.0" friction="1.0" />
-			<limit effort="10" velocity="${M_PI / 2.0}" lower="0" upper="${joint_2_limit}"/>
-                        <safety_controller k_position="20" k_velocity="25" soft_lower_limit="${threshold}" soft_upper_limit="${joint_2_limit_soft}" />
-=======
 			<dynamics damping="1" friction="1" />
 			<limit effort="${9.5}" velocity="${M_PI / 2.0}" lower="0" upper="${joint_2_limit}"/>
                         <safety_controller k_position="20" k_velocity="${2*9.5/M_PI}" soft_lower_limit="${threshold}" soft_upper_limit="${joint_2_limit_soft}" />
->>>>>>> working
 		</joint>
 		<link name="${name}_link_2">
@@ -133,10 +114,4 @@
 			<child link="${name}_link_3"/>
 			<axis xyz="0 1 0"/>
-<<<<<<< HEAD
-			<!--<calibration rising="${arm_3_ref}" falling="${arm_3_ref}"/>-->
-			<dynamics damping="1.0" friction="1.0" />
-			<limit effort="10" velocity="${M_PI / 2.0}" lower="-${joint_3_limit}" upper="0"/>
-                        <safety_controller k_position="20" k_velocity="25" soft_lower_limit="-${joint_3_limit_soft}" soft_upper_limit="${threshold}" />
-=======
 			<dynamics damping="1" friction="1" />
 			<limit effort="${6}" velocity="${M_PI / 2.0}" lower="-${joint_3_limit}" upper="0"/>
@@ -151,5 +126,4 @@
 			<limit effort="${6}" velocity="${M_PI / 2.0}" lower="0" upper="${joint_3_limit}"/>
                         <safety_controller k_position="20" k_velocity="50" soft_lower_limit="${threshold}" soft_upper_limit="${joint_3_limit_soft}" />
->>>>>>> working
 		</joint>
 		<link name="${name}_link_3">
@@ -181,13 +155,7 @@
 			<axis xyz="0 1 0" />
 			<!--<calibration rising="${arm_4_ref}" falling="${arm_4_ref}"/>-->
-<<<<<<< HEAD
-			<dynamics damping="1.0" friction="1.0" />
-			<limit effort="10" velocity="${M_PI / 2.0}" lower="0" upper="${joint_4_limit}"/>
-			<safety_controller k_position="20" k_velocity="25" soft_lower_limit="0" soft_upper_limit="${joint_4_limit_soft}" />
-=======
 			<dynamics damping="1" friction="1" />
 			<limit effort="${2}" velocity="${M_PI / 2.0}" lower="0" upper="${joint_4_limit}"/>
 			<safety_controller k_position="20" k_velocity="100" soft_lower_limit="0" soft_upper_limit="${joint_4_limit_soft}" />
->>>>>>> working
 		</joint>
 		<link name="${name}_link_4">
@@ -219,13 +187,7 @@
 			<axis xyz="0 0 -1" />
 			<!--<calibration rising="${arm_5_ref}" falling="${arm_5_ref}"/>-->
-<<<<<<< HEAD
-			<dynamics damping="1.0" friction="1.0" />
-			<limit effort="10" velocity="${M_PI / 2.0}" lower="0" upper="${joint_5_limit}" />
-                        <safety_controller k_position="20" k_velocity="25" soft_lower_limit="0" soft_upper_limit="${joint_5_limit_soft}" />
-=======
 			<dynamics damping="1" friction="1" />
 			<limit effort="1" velocity="${M_PI / 2.0}" lower="0" upper="${joint_5_limit}" />
                         <safety_controller k_position="20" k_velocity="100" soft_lower_limit="0" soft_upper_limit="${joint_5_limit_soft}" />
->>>>>>> working
 		</joint>
 		<link name="${name}_link_5">

File: youbot_common/youbot_description/urdf/youbot_arm/limits.urdf.xacro (robot description, xacro)
@@ -29,6 +29,4 @@
 	<property name="link_5_mass" value="0.1" />-->
 	<!-- TODO: add inertia tensor-->
-<<<<<<< HEAD
-=======
 	<xacro:macro name="default_origin">
         	<origin xyz="0 0 0" rpy="0 0 0"/> <!-- no data known -->
@@ -64,4 +62,3 @@
 		<inertia ixx="0.000280" ixy="0.000000" ixz="0.000000" iyy="0.000339" iyz="0.000000" izz="0.000119" />
 	</xacro:macro>
->>>>>>> working
 </robot>

Commit message: validation of the model with a real youbot. cleaning up

File: youbot_common/youbot_description/urdf/youbot_arm/arm.urdf.xacro (robot description, xacro)
@@ -122,8 +122,8 @@
 			<parent link="${name}_link_2"/>
 			<child link="${name}_link_3"/>
-			<axis xyz="0 -1 0"/>
-			<dynamics damping="1" friction="1" />
-			<limit effort="${6}" velocity="${M_PI / 2.0}" lower="0" upper="${joint_3_limit}"/>
-                        <safety_controller k_position="20" k_velocity="50" soft_lower_limit="${threshold}" soft_upper_limit="${joint_3_limit_soft}" />
+			<axis xyz="0 1 0"/>
+			<dynamics damping="1" friction="1" />
+			<limit effort="${6}" velocity="${M_PI / 2.0}" lower="-${joint_3_limit}" upper="0"/>
+                        <safety_controller k_position="20" k_velocity="50" soft_lower_limit="-${joint_3_limit_soft}" soft_upper_limit="-${threshold}" />
 		</joint>
 		<link name="${name}_link_3">

Commit message: urdf/arm: remove offsets for arm joints, use geometrical zeros
Signed-off-by: Ruben Smits <ruben.smits@mech.kuleuven.be>

File: youbot_common/youbot_description/urdf/youbot_arm/arm.urdf.xacro (robot description, xacro)
@@ -39,8 +39,8 @@
 		<!-- joint between arm_0_link and arm_1_link -->
 		<joint name="${name}_joint_1" type="revolute">
-			<origin xyz="0.024 0 0.096" rpy="0 0 ${170 * M_PI / 180}"/>
+			<origin xyz="0.024 0 0.096" rpy="0 0 0"/>
 			<parent link="${name}_link_0"/>
 			<child link="${name}_link_1"/>
-			<axis xyz="0 0 -1"/>
+			<axis xyz="0 0 1"/>
 			<!--<calibration rising="${arm_1_ref}" falling="${arm_1_ref}"/>-->
 			<dynamics damping="1.0" friction="1.0" />
@@ -73,8 +73,8 @@
 		<!-- joint between arm_1_link and arm_2_link -->
 		<joint name="${name}_joint_2" type="revolute">
-			<origin xyz="0.033 0 0.019" rpy="0 ${-65 * M_PI / 180} 0"/>
+			<origin xyz="0.033 0 0.019" rpy="0 0 0"/>
 			<parent link="${name}_link_1"/>
 			<child link="${name}_link_2"/>
-			<axis xyz="0 1 0"/>
+			<axis xyz="0 -1 0"/>
 			<!--<calibration rising="${arm_2_ref}" falling="${arm_2_ref}"/>-->
 			<dynamics damping="1.0" friction="1.0" />
@@ -107,5 +107,5 @@
 		<!-- joint between arm_2_link and arm_3_link -->
 		<joint name="${name}_joint_3" type="revolute">
-			<origin xyz="0.000 0.000 0.155" rpy="0 ${146 * M_PI / 180} 0"/>
+			<origin xyz="0.000 0.000 0.155" rpy="0 0 0"/>
 			<parent link="${name}_link_2"/>
 			<child link="${name}_link_3"/>
@@ -141,8 +141,8 @@
 		<!-- joint between arm_3_link and arm_4_link -->
 		<joint name="${name}_joint_4" type="revolute">
-			<origin xyz="0.000 0.000 0.135" rpy="0 ${-102.5 * M_PI / 180} 0" />
+			<origin xyz="0.000 0.000 0.135" rpy="0 0 0" />
 			<parent link="${name}_link_3"/>
 			<child link="${name}_link_4"/>
-			<axis xyz="0 1 0" />
+			<axis xyz="0 -1 0" />
 			<!--<calibration rising="${arm_4_ref}" falling="${arm_4_ref}"/>-->
 			<dynamics damping="1.0" friction="1.0" />
@@ -175,5 +175,5 @@
 		<!-- joint between arm_4_link and arm_5_link -->
 		<joint name="${name}_joint_5" type="revolute">
-			<origin xyz="-0.002 0 0.130" rpy="0 0 ${167.5 * M_PI / 180}" />
+			<origin xyz="-0.002 0 0.130" rpy="0 0 0" />
 			<parent link="${name}_link_4"/>
 			<child link="${name}_link_5"/>
