Commit message: model update

File: youbot_common/youbot_description/urdf/youbot_arm/arm.gazebo.xacro (robot description, xacro)
@@ -14,17 +14,17 @@
 		</gazebo>
 		<gazebo reference="${name}_link_2">
-			<material value="youbot/Orange" />
+			<!--<material value="youbot/Orange" />-->
 			<turnGravityOff>false</turnGravityOff>
 		</gazebo>
 		<gazebo reference="${name}_link_3">
-			<material value="youbot/Orange" />
+			<!--<material value="youbot/Orange" />-->
 			<turnGravityOff>false</turnGravityOff>
 		</gazebo>
 		<gazebo reference="${name}_link_4">
-			<material value="youbot/Orange" />
+			<!--<material value="youbot/Orange" />-->
 			<turnGravityOff>false</turnGravityOff>
 		</gazebo>
 		<gazebo reference="${name}_link_5">
-			<material value="youbot/DarkGrey" />
+			<!--<material value="youbot/DarkGrey" />-->
 			<turnGravityOff>false</turnGravityOff>
 		</gazebo>

File: youbot_common/youbot_description/urdf/youbot_arm/arm.urdf.xacro (robot description, xacro)
@@ -90,7 +90,7 @@
 			</inertial>
 			<visual>
-			<origin xyz="0.000 0.000 0.000" rpy="0 0 0" />
-				<geometry>
-					<mesh filename="package://youbot_description/meshes/youbot_arm/arm2.stl" />
+			<origin xyz="0 -0.032 0.078" rpy="0 0 0" />
+				<geometry>
+					<mesh filename="package://youbot_description/meshes/youbot_arm/arm2.dae" />
 				</geometry>
 				<material name="Orange" />
@@ -124,7 +124,7 @@
 			</inertial>
 			<visual>
-				<origin xyz="0 0 0" rpy="0 0 0" />
-				<geometry>
-					<mesh filename="package://youbot_description/meshes/youbot_arm/arm3.stl" />
+				<origin xyz="0.000 0.028 0.079" rpy="0 0 0" />
+				<geometry>
+					<mesh filename="package://youbot_description/meshes/youbot_arm/arm3.dae" />
 				</geometry>
 				<material name="Orange" />
@@ -158,7 +158,7 @@
 			</inertial>
 			<visual>
-				<origin xyz="0 0 0" rpy="0 0 0" />
-				<geometry>
-					<mesh filename="package://youbot_description/meshes/youbot_arm/arm4.stl" />
+				<origin xyz="0 -0.010 0.029" rpy="0 0 0"/>
+				<geometry>
+					<mesh filename="package://youbot_description/meshes/youbot_arm/arm4.dae" />
 				</geometry>
 				<material name="Orange" />
@@ -186,12 +186,12 @@
 		<link name="${name}_link_5">
 			<inertial>
-				<origin xyz="0.03 0 -0.030" rpy="0 0 0" />
+				<origin xyz="0.003 0 -0.034" rpy="0 0 0" />
 				<mass value="${link_5_mass}"/>
 				<inertia ixx="0.01" ixy="0" ixz="0" iyy="0.01" iyz="0" izz="0.01" />
 			</inertial>
 			<visual>
-				<origin xyz="0 0 0" rpy="0 0 0" />
-				<geometry>
-					<mesh filename="package://youbot_description/meshes/youbot_arm/arm5.stl" />
+				<origin xyz="0.003 0 -0.034" rpy="0 0 0" />
+				<geometry>
+					<mesh filename="package://youbot_description/meshes/youbot_arm/arm5.dae" />
 				</geometry>
 				<material name="DarkGrey" />

File: youbot_common/youbot_description/urdf/youbot_base/base.urdf.xacro (robot description, xacro)
@@ -4,4 +4,6 @@
         xmlns:interface="http://playerstage.sourceforge.net/gazebo/xmlschema/#interface"
         xmlns:xacro="http://ros.org/wiki/xacro">
+	<!-- sensors -->
+	<include filename="$(find youbot_description)/urdf/sensors/hokuyo_urg04_laser.urdf.xacro"/>
 	<include filename="$(find youbot_description)/urdf/youbot_base/base.gazebo.xacro" />
 	<include filename="$(find youbot_description)/urdf/youbot_base/base.transmission.xacro" />
@@ -80,4 +82,8 @@
       			</collision>
     		</link>
+		<!-- base laser front -->
+    		<xacro:hokuyo_urg04_laser name="${name}_laser_front" parent="${name}" ros_topic="scan_front" update_rate="10" min_angle="-2.09" max_angle="2.09" >
+     			 <origin xyz="0.3 0 -0.03" rpy="0 0 0" />
+    		</xacro:hokuyo_urg04_laser>
 	<!-- front left wheel -->
 		<joint name="caster_joint_fl" type="continuous">

Commit message: patches to get velocity controller working
Signed-off-by: Steven Bellens <steven.bellens@mech.kuleuven.be>
Signed-off-by: Tinne De Laet <Tinne.DeLaet@mech.kuleuven.be>

File: youbot_common/youbot_description/urdf/youbot_arm/arm.gazebo.xacro (robot description, xacro)
@@ -7,25 +7,25 @@
 		<gazebo reference="${name}_link_0">
 			<material value="youbot/DarkGrey" />
-			<turnGravityOff>false</turnGravityOff>
+			<turnGravityOff>true</turnGravityOff>
 		</gazebo>
 		<gazebo reference="${name}_link_1">
 			<!--<material value="youbot/Orange" />-->
-			<turnGravityOff>false</turnGravityOff>
+			<turnGravityOff>true</turnGravityOff>
 		</gazebo>
 		<gazebo reference="${name}_link_2">
 			<!--<material value="youbot/Orange" />-->
-			<turnGravityOff>false</turnGravityOff>
+			<turnGravityOff>true</turnGravityOff>
 		</gazebo>
 		<gazebo reference="${name}_link_3">
 			<!--<material value="youbot/Orange" />-->
-			<turnGravityOff>false</turnGravityOff>
+			<turnGravityOff>true</turnGravityOff>
 		</gazebo>
 		<gazebo reference="${name}_link_4">
 			<!--<material value="youbot/Orange" />-->
-			<turnGravityOff>false</turnGravityOff>
+			<turnGravityOff>true</turnGravityOff>
 		</gazebo>
 		<gazebo reference="${name}_link_5">
 			<!--<material value="youbot/DarkGrey" />-->
-			<turnGravityOff>false</turnGravityOff>
+			<turnGravityOff>true</turnGravityOff>
 		</gazebo>
 	</xacro:macro>

File: youbot_common/youbot_description/urdf/youbot_arm/arm.urdf.xacro (robot description, xacro)
@@ -39,24 +39,19 @@
 		<!-- joint between arm_0_link and arm_1_link -->
 		<joint name="${name}_joint_1" type="revolute">
-			<origin xyz="0.024 0 0.096" rpy="0 0 ${170 * M_PI / 180}"/>
+			<origin xyz="0.024 0 0.096" rpy="0 0 0"/>
 			<parent link="${name}_link_0"/>
 			<child link="${name}_link_1"/>
-			<axis xyz="0 0 -1"/>
+			<axis xyz="0 0 1"/>
 			<!--<calibration rising="${arm_1_ref}" falling="${arm_1_ref}"/>-->
-			<dynamics damping="1" friction="1" />
-			<!-- damping - N*s/m, N*s*m/rad -->
-			<!-- friction - N, N*m -->
-			<limit effort="${9.5}" velocity="${M_PI / 2.0}" lower="0" upper="${joint_1_limit}"/>
-			<!--effort - N, N*m-->
-			<!--velocity - m/s, rad/s-->
-			<safety_controller k_position="20" k_velocity="${9.5/M_PI / 2.0}" soft_lower_limit="${threshold}" soft_upper_limit="${joint_1_limit_soft}" />
-			<!--k_position N/m, N/rad-->
-			<!--k_velocity N*s/m, N*s*m/rad-->
-			<!--for details: http://www.ros.org/wiki/pr2_controller_manager/safety_limits-->
+			<dynamics damping="1.0" friction="1.0" />
+			<limit effort="10" velocity="${M_PI / 2.0}" lower="${joint_1_lower_limit}" upper="${joint_1_upper_limit}"/>
+			<safety_controller k_position="20" k_velocity="25" soft_lower_limit="${joint_1_lower_limit_soft}" soft_upper_limit="${joint_1_upper_limit_soft}" />
 		</joint>
 		<link name="${name}_link_1">
 			<inertial>
+				<!--<origin xyz="0 0 -0.003" rpy="0 0 0" />-->
+				<origin xyz="0 0 0" rpy="0 0 0" />
 				<mass value="${link_1_mass}"/>
-				<xacro:link_1_inertia_tensor />
+				<inertia ixx="0.01" ixy="0" ixz="0" iyy="0.01" iyz="0" izz="0.01" />
 			</inertial>
 			<visual>
@@ -78,28 +73,30 @@
 		<!-- joint between arm_1_link and arm_2_link -->
 		<joint name="${name}_joint_2" type="revolute">
-			<origin xyz="0.033 0 0.019" rpy="0 ${-65 * M_PI / 180} 0"/>
+			<origin xyz="0.033 0 0.019" rpy="0 0 0"/>
 			<parent link="${name}_link_1"/>
 			<child link="${name}_link_2"/>
-			<axis xyz="0 1 0"/>
+			<axis xyz="0 -1 0"/>
 			<!--<calibration rising="${arm_2_ref}" falling="${arm_2_ref}"/>-->
-			<dynamics damping="1" friction="1" />
-			<limit effort="${9.5}" velocity="${M_PI / 2.0}" lower="0" upper="${joint_2_limit}"/>
-                        <safety_controller k_position="20" k_velocity="${2*9.5/M_PI}" soft_lower_limit="${threshold}" soft_upper_limit="${joint_2_limit_soft}" />
+			<dynamics damping="1.0" friction="1.0" />
+			<limit effort="10" velocity="${M_PI / 2.0}" lower="${joint_2_lower_limit}" upper="${joint_2_upper_limit}"/>
+                        <safety_controller k_position="20" k_velocity="25" soft_lower_limit="${joint_2_lower_limit_soft}" soft_upper_limit="${joint_2_upper_limit_soft}" />
 		</joint>
 		<link name="${name}_link_2">
 			<inertial>
-				<mass value="${link_2_mass}"/>
-				<xacro:link_2_inertia_tensor />
-			</inertial>
-			<visual>
-			<origin xyz="0 -0.032 0.078" rpy="0 0 0" />
-				<geometry>
-					<mesh filename="package://youbot_description/meshes/youbot_arm/arm2.dae" />
-				</geometry>
-				<material name="Orange" />
-			</visual>
-			<collision>
 				<!--<origin xyz="0.001 -0.041 0.074" rpy="0 0 0" />-->
 				<origin xyz="0 -0.032 0.078" rpy="0 0 0" />
+				<mass value="${link_2_mass}"/>
+				<inertia ixx="0.01" ixy="0" ixz="0" iyy="0.01" iyz="0" izz="0.01" />
+			</inertial>
+			<visual>
+			<origin xyz="0 -0.032 0.078" rpy="0 0 0" />
+				<geometry>
+					<mesh filename="package://youbot_description/meshes/youbot_arm/arm2.dae" />
+				</geometry>
+				<material name="Orange" />
+			</visual>
+			<collision>
+				<!--<origin xyz="0.001 -0.041 0.074" rpy="0 0 0" />-->
+				<origin xyz="0 -0.032 0.078" rpy="0 0 0" />
 				<geometry>
 					<mesh filename="package://youbot_description/meshes/youbot_arm/arm2_convex.stl" />
@@ -109,37 +106,31 @@
 		</link>
 		<!-- joint between arm_2_link and arm_3_link -->
-		<!--<joint name="${name}_joint_3" type="revolute">
-			<origin xyz="0.000 0.000 0.155" rpy="0 ${146 * M_PI / 180} 0"/>
+		<joint name="${name}_joint_3" type="revolute">
+			<origin xyz="0.000 0.000 0.155" rpy="0 0 0"/>
 			<parent link="${name}_link_2"/>
 			<child link="${name}_link_3"/>
 			<axis xyz="0 1 0"/>
-			<dynamics damping="1" friction="1" />
-			<limit effort="${6}" velocity="${M_PI / 2.0}" lower="-${joint_3_limit}" upper="0"/>
-                        <safety_controller k_position="20" k_velocity="50" soft_lower_limit="-${joint_3_limit_soft}" soft_upper_limit="${threshold}" />
-		</joint>-->
-		<joint name="${name}_joint_3" type="revolute">
-			<origin xyz="0.000 0.000 0.155" rpy="0 ${146 * M_PI / 180} 0"/>
-			<parent link="${name}_link_2"/>
-			<child link="${name}_link_3"/>
-			<axis xyz="0 1 0"/>
-			<dynamics damping="1" friction="1" />
-			<limit effort="${6}" velocity="${M_PI / 2.0}" lower="-${joint_3_limit}" upper="0"/>
-                        <safety_controller k_position="20" k_velocity="50" soft_lower_limit="-${joint_3_limit_soft}" soft_upper_limit="-${threshold}" />
+			<!--<calibration rising="${arm_3_ref}" falling="${arm_3_ref}"/>-->
+			<dynamics damping="1.0" friction="1.0" />
+			<limit effort="10" velocity="${M_PI / 2.0}" lower="${joint_3_lower_limit}" upper="${joint_3_upper_limit}"/>
+                        <safety_controller k_position="20" k_velocity="25" soft_lower_limit="${joint_3_lower_limit_soft}" soft_upper_limit="${joint_3_upper_limit_soft}" />
 		</joint>
 		<link name="${name}_link_3">
 			<inertial>
-				<mass value="${link_3_mass}"/>
-				<xacro:link_3_inertia_tensor />
-			</inertial>
-			<visual>
-				<origin xyz="0.000 0.028 0.079" rpy="0 0 0" />
-				<geometry>
-					<mesh filename="package://youbot_description/meshes/youbot_arm/arm3.dae" />
-				</geometry>
-				<material name="Orange" />
-			</visual>
-			<collision>
 				<!--<origin xyz="0.000 0.025 0.067" rpy="0 0 0" />-->
 				<origin xyz="0.000 0.028 0.079" rpy="0 0 0" />
+				<mass value="${link_3_mass}"/>
+				<inertia ixx="0.01" ixy="0" ixz="0" iyy="0.01" iyz="0" izz="0.01" />
+			</inertial>
+			<visual>
+				<origin xyz="0.000 0.028 0.079" rpy="0 0 0" />
+				<geometry>
+					<mesh filename="package://youbot_description/meshes/youbot_arm/arm3.dae" />
+				</geometry>
+				<material name="Orange" />
+			</visual>
+			<collision>
+				<!--<origin xyz="0.000 0.025 0.067" rpy="0 0 0" />-->
+				<origin xyz="0.000 0.028 0.079" rpy="0 0 0" />
 				<geometry>
 					<mesh filename="package://youbot_description/meshes/youbot_arm/arm3_convex.stl" />
@@ -150,17 +141,19 @@
 		<!-- joint between arm_3_link and arm_4_link -->
 		<joint name="${name}_joint_4" type="revolute">
-			<origin xyz="0.000 0.000 0.135" rpy="0 ${-102.5 * M_PI / 180} 0" />
+			<origin xyz="0.000 0.000 0.135" rpy="0 0 0" />
 			<parent link="${name}_link_3"/>
 			<child link="${name}_link_4"/>
-			<axis xyz="0 1 0" />
+			<axis xyz="0 -1 0" />
 			<!--<calibration rising="${arm_4_ref}" falling="${arm_4_ref}"/>-->
-			<dynamics damping="1" friction="1" />
-			<limit effort="${2}" velocity="${M_PI / 2.0}" lower="0" upper="${joint_4_limit}"/>
-			<safety_controller k_position="20" k_velocity="100" soft_lower_limit="0" soft_upper_limit="${joint_4_limit_soft}" />
+			<dynamics damping="1.0" friction="1.0" />
+			<limit effort="10" velocity="${M_PI / 2.0}" lower="${joint_4_lower_limit}" upper="${joint_4_upper_limit}"/>
+			<safety_controller k_position="20" k_velocity="25" soft_lower_limit="${joint_4_lower_limit_soft}" soft_upper_limit="${joint_4_upper_limit_soft}" />
 		</joint>
 		<link name="${name}_link_4">
 			<inertial>
+				<!--<origin xyz="0 0 0.026" rpy="0 0 0"/>-->
+				<origin xyz="0 -0.010 0.029" rpy="0 0 0"/>
 				<mass value="${link_4_mass}"/>
-				<xacro:link_4_inertia_tensor />
+				<inertia ixx="0.01" ixy="0" ixz="0" iyy="0.01" iyz="0" izz="0.01" />
 			</inertial>
 			<visual>
@@ -182,17 +175,18 @@
 		<!-- joint between arm_4_link and arm_5_link -->
 		<joint name="${name}_joint_5" type="revolute">
-			<origin xyz="-0.002 0 0.130" rpy="0 0 ${167.5 * M_PI / 180}" />
+			<origin xyz="-0.002 0 0.130" rpy="0 0 0" />
 			<parent link="${name}_link_4"/>
 			<child link="${name}_link_5"/>
-			<axis xyz="0 0 -1" />
+			<axis xyz="0 0 1" />
 			<!--<calibration rising="${arm_5_ref}" falling="${arm_5_ref}"/>-->
-			<dynamics damping="1" friction="1" />
-			<limit effort="1" velocity="${M_PI / 2.0}" lower="0" upper="${joint_5_limit}" />
-                        <safety_controller k_position="20" k_velocity="100" soft_lower_limit="0" soft_upper_limit="${joint_5_limit_soft}" />
+			<dynamics damping="1.0" friction="1.0" />
+			<limit effort="10" velocity="${M_PI / 2.0}" lower="${joint_5_lower_limit}" upper="${joint_5_upper_limit}" />
+                        <safety_controller k_position="20" k_velocity="25" soft_lower_limit="${joint_5_lower_limit_soft}" soft_upper_limit="${joint_5_upper_limit_soft}" />
 		</joint>
 		<link name="${name}_link_5">
 			<inertial>
+				<origin xyz="0.003 0 -0.034" rpy="0 0 0" />
 				<mass value="${link_5_mass}"/>
-				<xacro:link_5_inertia_tensor />
+				<inertia ixx="0.01" ixy="0" ixz="0" iyy="0.01" iyz="0" izz="0.01" />
 			</inertial>
 			<visual>

File: youbot_common/youbot_description/urdf/youbot_arm/limits.urdf.xacro (robot description, xacro)
@@ -5,14 +5,24 @@
         <property name="threshold" value="0.01" />
 	<!-- arm limits positions (deg) -->
-	<property name="joint_1_limit" value="${M_PI * (169 + 169) / 180}" />
-	<property name="joint_2_limit" value="${M_PI * (90 + 65) / 180}" />
-	<property name="joint_3_limit" value="${M_PI * (146 + 151) / 180}" />
-	<property name="joint_4_limit" value="${M_PI * (102.5 + 102.5) / 180}" />
-	<property name="joint_5_limit" value="${M_PI * (167.5 + 167.5) / 180}" />
-        <property name="joint_1_limit_soft" value="${M_PI * (169 + 169) / 180 - threshold}" />
-	<property name="joint_2_limit_soft" value="${M_PI * (90 + 65) / 180 - threshold}" />
-	<property name="joint_3_limit_soft" value="${M_PI * (146 + 151) / 180 - threshold}" />
-	<property name="joint_4_limit_soft" value="${M_PI * (102.5 + 102.5) / 180 - threshold}" />
-	<property name="joint_5_limit_soft" value="${M_PI * (167.5 + 167.5) / 180 - threshold}" />
+	<property name="joint_1_lower_limit" value="${M_PI * -170 / 180}" />
+	<property name="joint_1_upper_limit" value="${M_PI * 169 / 180}" />
+	<property name="joint_2_lower_limit" value="${M_PI * -90 / 180}" />
+	<property name="joint_2_upper_limit" value="${M_PI * 65 / 180}" />
+	<property name="joint_3_lower_limit" value="${M_PI * -151 / 180}" />
+	<property name="joint_3_upper_limit" value="${M_PI * 146 / 180}" />
+	<property name="joint_4_lower_limit" value="${M_PI * -102.5 / 180}" />
+	<property name="joint_4_upper_limit" value="${M_PI * 102.5 / 180}" />
+	<property name="joint_5_lower_limit" value="${M_PI * -167.5 / 180}" />
+	<property name="joint_5_upper_limit" value="${M_PI * 167.5 / 180}" />
+  <property name="joint_1_lower_limit_soft" value="${M_PI * -170 / 180 + threshold}" />
+  <property name="joint_1_upper_limit_soft" value="${M_PI * 169 / 180 - threshold}" />
+	<property name="joint_2_lower_limit_soft" value="${M_PI * -90 / 180 + threshold}" />
+	<property name="joint_2_upper_limit_soft" value="${M_PI * 65 / 180 - threshold}" />
+	<property name="joint_3_lower_limit_soft" value="${M_PI * -151 / 180 + threshold}" />
+	<property name="joint_3_upper_limit_soft" value="${M_PI * 146 / 180 - threshold}" />
+	<property name="joint_4_lower_limit_soft" value="${M_PI * -102.5 / 180 + threshold}" />
+	<property name="joint_4_upper_limit_soft" value="${M_PI * 102.5 / 180 - threshold}" />
+	<property name="joint_5_lower_limit_soft" value="${M_PI * -167.5 / 180 + threshold}" />
+	<property name="joint_5_upper_limit_soft" value="${M_PI * 167.5 / 180 - threshold}" />
 	<!-- dynamic properties : mass (kg) Alu data sheet -->
 	<property name="link_0_mass" value="0.845" />

File: youbot_common/youbot_description/urdf/youbot_gripper/gripper.gazebo.xacro (robot description, xacro)
@@ -7,16 +7,16 @@
 		<gazebo reference="${name}_palm_link">
 			<material>Gazebo/Black</material>
-			<turnGravityOff>false</turnGravityOff>
-			<selfCollide>true</selfCollide>
+			<turnGravityOff>true</turnGravityOff>
+			<selfCollide>false</selfCollide>
 		</gazebo>
-		<gazebo reference="${name}_finger_l_link">
+		<gazebo reference="${name}_finger_link_l">
 			<material>Gazebo/Black</material>
-			<turnGravityOff>false</turnGravityOff>
-			<selfCollide>true</selfCollide>
+			<turnGravityOff>true</turnGravityOff>
+			<selfCollide>false</selfCollide>
 		</gazebo>
-		<gazebo reference="${name}_finger_r_link">
+		<gazebo reference="${name}_finger_link_r">
 			<material>Gazebo/Black</material>
-			<turnGravityOff>false</turnGravityOff>
-			<selfCollide>true</selfCollide>
+			<turnGravityOff>true</turnGravityOff>
+			<selfCollide>false</selfCollide>
 		</gazebo>
 	</xacro:macro>
