Commit message: add base joints

File: youbot_common/youbot_description/robots/youbot.urdf.xacro (robot description, xacro)
@@ -33,5 +33,5 @@
     <origin xyz="-0.159 0 0.046" rpy="0 0 0" />
   </xacro:youbot_plate>
-  <xacro:youbot_arm name="arm" parent="base_link">
+  <xacro:youbot_arm name="arm" parent="base_to_arm_link">
     <origin xyz="0.143 0 0.046" rpy="0 0 0" />
   </xacro:youbot_arm>

File: youbot_common/youbot_description/urdf/youbot_base/base.urdf.xacro (robot description, xacro)
@@ -82,4 +82,64 @@
       			</collision>
     		</link>
+		<!-- base_link -> base_rot_joint -> base_x_link  -->
+		<joint name="${name}_rot_joint" type="revolute">
+			<origin xyz="0 0 0" rpy="0 0 0"/>
+			<parent link="${name}_link"/>
+			<child link="${name}_x_link"/>
+			<axis xyz="0 0 1"/>
+			<!--<calibration rising="${arm_1_ref}" falling="${arm_1_ref}"/>-->
+			<!-- <dynamics damping="1.0" friction="1.0" /> -->
+			<limit effort="10" velocity="${M_PI / 2.0}" />
+			<!-- <safety_controller k_position="20" k_velocity="25" soft_lower_limit="${threshold}" soft_upper_limit="${joint_1_limit_soft}" /> -->
+		</joint>
+		<!-- base_x_link -->
+		<link name="${name}_x_link">
+      		  <inertial>
+		    <mass value="0.01" />
+		    <origin xyz="0 0 0" />
+		    <inertia ixx="1" ixy="0" ixz="0"
+			     iyy="1" iyz="0" izz="1" />
+      		  </inertial>
+    		</link>
+		<!-- base_x_link -> base_x_joint -> base_x_link -->
+		<joint name="${name}_x_joint" type="prismatic">
+		  <origin xyz="0 0 0" rpy="0 0 0"/>
+		  <parent link="${name}_x_link"/>
+		  <child link="${name}_y_link"/>
+		  <axis xyz="1 0 0"/>
+		  <!--<calibration rising="${arm_1_ref}" falling="${arm_1_ref}"/>-->
+		  <!-- <dynamics damping="1.0" friction="1.0" /> -->
+		  <!-- <limit effort="10" velocity="${M_PI / 2.0}" lower="0" upper="${joint_1_limit}"/> -->
+		  <!-- <safety_controller k_position="20" k_velocity="25" soft_lower_limit="${threshold}" soft_upper_limit="${joint_1_limit_soft}" /> -->
+		</joint>
+		<!-- base_y_link -->
+		<link name="${name}_y_link">
+      		  <inertial>
+		    <mass value="0.01" />
+		    <origin xyz="0 0 0" />
+		    <inertia ixx="1" ixy="0" ixz="0"
+			     iyy="1" iyz="0" izz="1" />
+      		  </inertial>
+    		</link>
+		<!-- base_y_link -> base_y_joint -->
+		<joint name="${name}_y_joint" type="prismatic">
+		  <origin xyz="0 0 0" rpy="0 0 0"/>
+		  <parent link="${name}_y_link"/>
+		  <child link="${name}_to_arm_link"/>
+		  <axis xyz="0 1 0"/>
+		  <!--<calibration rising="${arm_1_ref}" falling="${arm_1_ref}"/>-->
+		  <!-- <dynamics damping="1.0" friction="1.0" /> -->
+		  <!-- <limit effort="10" velocity="${M_PI / 2.0}" lower="0" upper="${joint_1_limit}"/> -->
+		  <!-- <safety_controller k_position="20" k_velocity="25" soft_lower_limit="${threshold}" soft_upper_limit="${joint_1_limit_soft}" /> -->
+		</joint>
+		<!-- base_to_arm_link -->
+		<link name="${name}_to_arm_link">
+      		  <inertial>
+		    <mass value="0.01" />
+		    <origin xyz="0 0 0" />
+		    <inertia ixx="1" ixy="0" ixz="0"
+			     iyy="1" iyz="0" izz="1" />
+      		  </inertial>
+    		</link>
 		<!-- base laser front -->
     		<xacro:hokuyo_urg04_laser name="${name}_laser_front" parent="${name}" ros_topic="scan_front" update_rate="10" min_angle="-2.09" max_angle="2.09" >
