Commit message: urdf/gripper: make fingers fixed until we have a service for the gripper and increase the grippers mass
Signed-off-by: Ruben Smits <ruben.smits@mech.kuleuven.be>

File: youbot_common/youbot_description/urdf/youbot_gripper/gripper.urdf.xacro (robot description, xacro)
@@ -17,5 +17,5 @@
 			<inertial>
 				<origin xyz="0 0 0" rpy="0 0 0"/>
-				<mass value="0.1"/>
+				<mass value="0.75"/>
 				<inertia ixx="0.01" ixy="0" ixz="0" iyy="0.01" iyz="0" izz="0.01" />
 			</inertial>
@@ -35,5 +35,5 @@
 			</collision>
 		</link>
-		<joint name="${name}_finger_joint_l" type="prismatic">
+		<joint name="${name}_finger_joint_l" type="fixed">
 			<origin xyz="0.004 0.008 0.046" rpy="0 0 ${M_PI}" />
 			<parent link="${name}_palm_link"/>
@@ -65,5 +65,5 @@
 			</collision>
 		</link>
-               <joint name="${name}_finger_joint_r" type="prismatic">
+               <joint name="${name}_finger_joint_r" type="fixed">
 			<origin xyz="0.004 -0.008 0.046" rpy="0 0 0" />
 			<parent link="${name}_palm_link"/>

Commit message: replace stl with dae files to also see the gripper in rviz

File: youbot_common/youbot_description/urdf/youbot_gripper/gripper.urdf.xacro (robot description, xacro)
@@ -23,5 +23,5 @@
 				<origin xyz="0 0 0" rpy="0 0 0" />
 				<geometry>
-					<mesh filename="package://youbot_description/meshes/youbot_gripper/palm.stl" />
+					<mesh filename="package://youbot_description/meshes/youbot_gripper/palm.dae" />
 				</geometry>
 				<material name="DarkGrey" />
@@ -53,5 +53,5 @@
 				<origin xyz="0 0 0" rpy="0 0 0" />
 				<geometry>
-					<mesh filename="package://youbot_description/meshes/youbot_gripper/finger.stl" />
+					<mesh filename="package://youbot_description/meshes/youbot_gripper/finger.dae" />
 				</geometry>
 				<material name="DarkGrey" />
@@ -83,5 +83,5 @@
 				<origin xyz="0 0 0" rpy="0 0 0" />
 				<geometry>
-					<mesh filename="package://youbot_description/meshes/youbot_gripper/finger.stl" />
+					<mesh filename="package://youbot_description/meshes/youbot_gripper/finger.dae" />
 				</geometry>
 				<material name="DarkGrey" />
