Commit message: replace stl with dae files

File: youbot_common/youbot_description/tests/youbot_arm.urdf (robot description, URDF)
Before this commit: robot youbot, 10 links, 9 joints
Links:
- link gripper_finger_link_l: geometry collision mesh filename=package://youbot_description/meshes/youbot_gripper/finger_c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; visual mesh filename=package://youbot_description/meshes/youbot_gripper/finger.d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
- link gripper_finger_link_r: geometry collision mesh filename=package://youbot_description/meshes/youbot_gripper/finger_c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; visual mesh filename=package://youbot_description/meshes/youbot_gripper/finger.d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
- link gripper_palm_link: geometry collision mesh filename=package://youbot_description/meshes/youbot_gripper/palm_con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; visual mesh filename=package://youbot_description/meshes/youbot_gripper/palm.dae

File: youbot_common/youbot_description/tests/youbot_base.urdf (robot description, URDF)
Before this commit: robot youbot, 11 links, 10 joints
Links:
- link base_laser_front_link: geometry collision mesh filename=package://youbot_description/meshes/sensors/hokuyo_convex.d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; visual mesh filename=package://youbot_description/meshes/sensors/hokuyo.dae

File: youbot_common/youbot_description/tests/youbot_gripper.urdf (robot description, URDF)
Before this commit: robot youbot, 4 links, 3 joints
Links:
- link gripper_finger_link_l: geometry collision mesh filename=package://youbot_description/meshes/youbot_gripper/finger_c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; visual mesh filename=package://youbot_description/meshes/youbot_gripper/finger.d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
- link gripper_finger_link_r: geometry collision mesh filename=package://youbot_description/meshes/youbot_gripper/finger_c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; visual mesh filename=package://youbot_description/meshes/youbot_gripper/finger.d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
- link gripper_palm_link: geometry collision mesh filename=package://youbot_description/meshes/youbot_gripper/palm_con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; visual mesh filename=package://youbot_description/meshes/youbot_gripper/palm.dae

File: youbot_common/youbot_description/urdf/sensors/hokuyo_urg04_laser.urdf.xacro (robot description, xacro)
@@ -28,5 +28,5 @@
 		<origin xyz="0 0 0" rpy="0 0 0" />
 		<geometry>
-			<mesh filename="package://youbot_description/meshes/sensors/hokuyo_convex.stl" />
+			<mesh filename="package://youbot_description/meshes/sensors/hokuyo_convex.dae" />
 		</geometry>
 	</collision>

File: youbot_common/youbot_description/urdf/youbot_arm/arm.urdf.xacro (robot description, xacro)
@@ -32,5 +32,5 @@
 				<origin xyz="0 0 0" rpy="0 0 0"/>
 				<geometry>
-					<mesh filename="package://youbot_description/meshes/youbot_arm/arm0_convex.stl" />
+					<mesh filename="package://youbot_description/meshes/youbot_arm/arm0_convex.dae" />
 					<!--<cylinder length="0.078" radius="0.093"/>-->
 				</geometry>
@@ -71,5 +71,5 @@
 				<origin xyz="0 0 0" rpy="0 0 0" />
 				<geometry>
-					<mesh filename="package://youbot_description/meshes/youbot_arm/arm1_convex.stl" />
+					<mesh filename="package://youbot_description/meshes/youbot_arm/arm1_convex.dae" />
 					<!--<cylinder length="0.102" radius="0.080"/>-->
 				</geometry>
@@ -103,5 +103,5 @@
 				<origin xyz="0 -0.032 0.078" rpy="0 0 0" />
 				<geometry>
-					<mesh filename="package://youbot_description/meshes/youbot_arm/arm2_convex.stl" />
+					<mesh filename="package://youbot_description/meshes/youbot_arm/arm2_convex.dae" />
 					<!--<box size="0.074 0.082 0.222"/>-->
 				</geometry>
@@ -143,5 +143,5 @@
 				<origin xyz="0.000 0.028 0.079" rpy="0 0 0" />
 				<geometry>
-					<mesh filename="package://youbot_description/meshes/youbot_arm/arm3_convex.stl" />
+					<mesh filename="package://youbot_description/meshes/youbot_arm/arm3_convex.dae" />
 					<!--<box size="0.064 0.054 0.192"/>-->
 				</geometry>
@@ -175,5 +175,5 @@
 				<origin xyz="0 -0.010 0.029" rpy="0 0 0"/>
 				<geometry>
-					<mesh filename="package://youbot_description/meshes/youbot_arm/arm4_convex.stl" />
+					<mesh filename="package://youbot_description/meshes/youbot_arm/arm4_convex.dae" />
 					<!--<box size="0.058 0.100 0.118"/>-->
 				</geometry>
@@ -206,5 +206,5 @@
 				<origin xyz="0.003 0 -0.034" rpy="0 0 0" />
 				<geometry>
-					<mesh filename="package://youbot_description/meshes/youbot_arm/arm5_convex.stl" />
+					<mesh filename="package://youbot_description/meshes/youbot_arm/arm5_convex.dae" />
 					<!--<box size="0.054 0.096 0.030"/>-->
 				</geometry>

File: youbot_common/youbot_description/urdf/youbot_base/base.urdf.xacro (robot description, xacro)
@@ -78,5 +78,5 @@
         			<geometry>
           				<!--<box size="${base_size_x} ${base_size_y} ${base_size_z}" />-->
-					<mesh filename="package://youbot_description/meshes/youbot_base/base_convex.stl"/>
+					<mesh filename="package://youbot_description/meshes/youbot_base/base_convex.dae"/>
 	       			</geometry>
       			</collision>

File: youbot_common/youbot_description/urdf/youbot_gripper/gripper.urdf.xacro (robot description, xacro)
@@ -25,5 +25,5 @@
 					<mesh filename="package://youbot_description/meshes/youbot_gripper/palm.dae" />
 				</geometry>
-				<material name="DarkGrey" />
+				<material name="Black" />
 			</visual>
 			<collision>
@@ -31,5 +31,5 @@
 				<geometry>
 					<!--<box size="0.050 0.094 0.054"/>-->
-					<mesh filename="package://youbot_description/meshes/youbot_gripper/palm_convex.stl" />
+					<mesh filename="package://youbot_description/meshes/youbot_gripper/palm_convex.dae" />
 				</geometry>
 			</collision>
@@ -55,5 +55,5 @@
 					<mesh filename="package://youbot_description/meshes/youbot_gripper/finger.dae" />
 				</geometry>
-				<material name="DarkGrey" />
+				<material name="Black" />
 			</visual>
 			<collision>
@@ -61,5 +61,5 @@
 				<geometry>
 					<!--<box size="0.014 0.020 0.046"/>-->
-					<mesh filename="package://youbot_description/meshes/youbot_gripper/finger_convex.stl" />
+					<mesh filename="package://youbot_description/meshes/youbot_gripper/finger_convex.dae" />
 				</geometry>
 			</collision>
@@ -85,5 +85,5 @@
 					<mesh filename="package://youbot_description/meshes/youbot_gripper/finger.dae" />
 				</geometry>
-				<material name="DarkGrey" />
+				<material name="Black" />
 			</visual>
 			<collision>
@@ -91,5 +91,5 @@
 				<geometry>
 					<!--<box size="0.014 0.020 0.046"/>-->
-					<mesh filename="package://youbot_description/meshes/youbot_gripper/finger_convex.stl" />
+					<mesh filename="package://youbot_description/meshes/youbot_gripper/finger_convex.dae" />
 				</geometry>
 			</collision>

File: youbot_common/youbot_description/urdf/youbot_plate/plate.urdf.xacro (robot description, xacro)
@@ -22,10 +22,10 @@
 					<mesh filename="package://youbot_description/meshes/youbot_plate/plate.dae" />
 				</geometry>
-				<material name="DarkGrey" />
+				<material name="DarkGrey"/>
 			</visual>
 			<collision>
 				<origin xyz="0 0 0" rpy="0 0 0" />
 				<geometry>
-					<mesh filename="package://youbot_description/meshes/youbot_plate/plate_convex.stl" />
+					<mesh filename="package://youbot_description/meshes/youbot_plate/plate_convex.dae" />
 				</geometry>
 			</collision>
