Commit message: urdf/base: make wheels fixed for now until the base_service publishes the jointstate of the wheels
Signed-off-by: Ruben Smits <ruben.smits@mech.kuleuven.be>

File: youbot_common/youbot_description/urdf/youbot_base/base.urdf.xacro (robot description, xacro)
@@ -87,5 +87,5 @@
     		</xacro:hokuyo_urg04_laser>
 	<!-- front left wheel -->
-		<joint name="caster_joint_fl" type="continuous">
+		<joint name="caster_joint_fl" type="fixed">
 			<origin xyz="${caster_offset_x} ${caster_offset_y} ${caster_offset_z}" rpy="0 0 0" />
       			<axis xyz="0 0 1" />
@@ -104,5 +104,5 @@
       			</inertial>
    		</link>
-		<joint name="wheel_joint_fl" type="continuous">
+		<joint name="wheel_joint_fl" type="fixed">
       			<axis xyz="0 1 0" />
       			<limit effort="${wheel_joint_effort}" velocity="${wheel_joint_velocity}"/>
@@ -136,5 +136,5 @@
     		</link>
 	<!-- front right wheel -->
-		<joint name="caster_joint_fr" type="continuous">
+		<joint name="caster_joint_fr" type="fixed">
 			<origin xyz="${caster_offset_x} ${-caster_offset_y} ${caster_offset_z}" rpy="0 0 0" />
       			<axis xyz="0 0 1" />
@@ -153,5 +153,5 @@
       				</inertial>
    		</link>
-		<joint name="wheel_joint_fr" type="continuous">
+		<joint name="wheel_joint_fr" type="fixed">
       			<axis xyz="0 1 0" />
       			<limit effort="${wheel_joint_effort}" velocity="${wheel_joint_velocity}"/>
@@ -185,5 +185,5 @@
     		</link>
 	<!-- back left wheel -->
-		<joint name="caster_joint_bl" type="continuous">
+		<joint name="caster_joint_bl" type="fixed">
 			<origin xyz="${-caster_offset_x} ${caster_offset_y} ${caster_offset_z}" rpy="0 0 0" />
       			<axis xyz="0 0 1" />
@@ -202,5 +202,5 @@
       				</inertial>
    		</link>
-		<joint name="wheel_joint_bl" type="continuous">
+		<joint name="wheel_joint_bl" type="fixed">
       			<axis xyz="0 1 0" />
       			<limit effort="10" velocity="10"/>
@@ -235,5 +235,5 @@
     		</link>
 	<!-- back right wheel -->
-		<joint name="caster_joint_br" type="continuous">
+		<joint name="caster_joint_br" type="fixed">
 			<origin xyz="${-caster_offset_x} ${-caster_offset_y} ${caster_offset_z}" rpy="0 0 0" />
       			<axis xyz="0 0 1" />
@@ -252,5 +252,5 @@
       				</inertial>
    		</link>
-		<joint name="wheel_joint_br" type="continuous">
+		<joint name="wheel_joint_br" type="fixed">
       			<axis xyz="0 1 0" />
       			<limit effort="${wheel_joint_effort}" velocity="${wheel_joint_velocity}"/>

Commit message: increase length of the wheels (represented as cylinder) for the collision model, since they were really thin

File: youbot_common/youbot_description/urdf/youbot_base/base.urdf.xacro (robot description, xacro)
@@ -131,5 +131,5 @@
         			<origin xyz="0 0 0" rpy="${M_PI/2} 0 0" />
         			<geometry>
-        		       		<cylinder radius="${wheel_radius}" length="${wheel_length}" />
+        		       		<cylinder radius="${wheel_radius}" length="${wheel_radius}" />
         	       		</geometry>
       			</collision>
@@ -180,5 +180,5 @@
         			<origin xyz="0 0 0" rpy="${M_PI/2} 0 0" />
         			<geometry>
-        		       		<cylinder radius="${wheel_radius}" length="${wheel_length}" />
+        		       		<cylinder radius="${wheel_radius}" length="${wheel_radius}" />
         	       		</geometry>
       			</collision>
@@ -230,5 +230,5 @@
         			<origin xyz="0 0 0" rpy="${M_PI/2} 0 0" />
         			<geometry>
-        		       		<cylinder radius="${wheel_radius}" length="${wheel_length}" />
+        		       		<cylinder radius="${wheel_radius}" length="${wheel_radius}" />
         	       		</geometry>
       			</collision>
@@ -279,5 +279,5 @@
         			<origin xyz="0 0 0" rpy="${M_PI/2} 0 0" />
         			<geometry>
-        		       		<cylinder radius="${wheel_radius}" length="${wheel_length}" />
+        		       		<cylinder radius="${wheel_radius}" length="${wheel_radius}" />
         	       		</geometry>
       			</collision>

Commit message: remove warning (interia not allowed in base_footprint) and drag base_footprint down to the ground

File: youbot_common/youbot_description/urdf/youbot_base/base.urdf.xacro (robot description, xacro)
@@ -35,26 +35,20 @@
 	<xacro:macro name="youbot_base" params="name">
 		<link name="${name}_footprint">
-      			<inertial>
-        			<mass value="0.1" />
+      			<visual>
+        			<origin xyz="0 0 0" rpy="0 0 0" />
+        			<geometry>
+          				<box size="0.001 0.001 0.001" />
+        			</geometry>
+               			<material name="Red" />
+      			</visual>
+      			<collision>
         			<origin xyz="0 0 ${-base_size_z / 2.0}" rpy="0 0 0" />
-        			<inertia ixx="1.0" ixy="0.0" ixz="0.0"
-                 			iyy="1.0" iyz="0.0" izz="1.0" />
-      				</inertial>
-      			<visual>
-        			<origin xyz="0 0 0" rpy="0 0 0" />
         			<geometry>
           				<box size="0.001 0.001 0.001" />
         			</geometry>
-               			<material name="Red" />
-      			</visual>
-      			<collision>
-        			<origin xyz="0 0 ${-base_size_z / 2.0}" rpy="0 0 0" />
-        			<geometry>
-          				<box size="0.001 0.001 0.001" />
-        			</geometry>
       			</collision>
     		</link>
     		<joint name="${name}_footprint_joint" type="fixed">
-      			<origin xyz="0 0 0" rpy="0 0 0" />
+      			<origin xyz="0 0 0.08" rpy="0 0 0" />
       			<child link="${name}_link" />
       			<parent link="${name}_footprint"/>
