Commit message: adapt XML Gazebo syntax in URDF files for Groovy

File: youbot_common/youbot_description/gazebo/gazebo.urdf.xacro (robot description, xacro)
@@ -4,10 +4,9 @@
        xmlns:interface="http://playerstage.sourceforge.net/gazebo/xmlschema/#interface">
   <gazebo>
-    <controller:gazebo_ros_controller_manager name="gazebo_ros_controller_manager" plugin="libgazebo_ros_controller_manager.so">
+    <plugin name="gazebo_ros_controller_manager" filename="libgazebo_ros_controller_manager.so">
       <alwaysOn>true</alwaysOn>
       <updateRate>1000.0</updateRate>
-      <interface:audio name="gazebo_ros_controller_manager_dummy_iface" />
-    </controller:gazebo_ros_controller_manager>
-    <controller:gazebo_ros_power_monitor name="gazebo_ros_power_monitor_controller" plugin="libgazebo_ros_power_monitor.so">
+    </plugin>
+    <plugin name="gazebo_ros_power_monitor_controller" filename="libgazebo_ros_power_monitor.so">
       <alwaysOn>true</alwaysOn>
       <updateRate>1.0</updateRate>
@@ -21,5 +20,5 @@
       <dischargeVoltage>15.52</dischargeVoltage>
       <chargeVoltage>16.41</chargeVoltage>
-    </controller:gazebo_ros_power_monitor>
+    </plugin>
   </gazebo>
 </robot>

File: youbot_common/youbot_description/urdf/sensors/hokuyo_urg04_laser.gazebo.xacro (robot description, xacro)
@@ -6,25 +6,32 @@
   <xacro:macro name="hokuyo_urg04_laser_gazebo" params="name ros_topic update_rate min_angle max_angle">
     <gazebo reference="${name}_link">
-      <sensor:ray name="${name}">
-        <rayCount>640</rayCount>
-        <rangeCount>640</rangeCount>
-        <laserCount>1</laserCount>
-        <origin>0.0 0.0 0.0</origin>
-        <displayRays>false</displayRays>
-        <minAngle>${min_angle*180.0/M_PI}</minAngle>
-        <maxAngle>${max_angle*180.0/M_PI}</maxAngle>
-        <minRange>0.05</minRange>
-        <maxRange>5.6</maxRange>
-        <resRange>0.36</resRange>
-        <updateRate>${update_rate}</updateRate>
-        <controller:gazebo_ros_laser name="gazebo_ros_${name}_controller" plugin="libgazebo_ros_laser.so">
-          <gaussianNoise>0.000</gaussianNoise>
-          <alwaysOn>true</alwaysOn>
-          <updateRate>${update_rate}</updateRate>
-          <topicName>${ros_topic}</topicName>
-          <frameName>/${name}_link</frameName>
-          <interface:laser name="gazebo_ros_${name}_iface" />
-        </controller:gazebo_ros_laser>
-      </sensor:ray>
+      <sensor name="${name}" type="ray">
+		<always_on>true</always_on>
+        <update_rate>${update_rate}</update_rate>
+		<pose>0 0 0 0 0 0</pose>
+		<visualize>false</visualize>
+        <ray>
+            <scan>
+                <horizontal>
+                    <samples>150</samples>
+                    <resolution>1.0</resolution>
+                    <min_angle>${min_angle}</min_angle>
+                    <max_angle>${max_angle}</max_angle>
+                </horizontal>
+            </scan>
+            <range>
+				<min>0.05</min>
+				<max>5.6</max>
+				<resolution>0.36</resolution>
+			</range>
+        </ray>
+        <plugin name="gazebo_ros_${name}_controller" filename="libgazebo_ros_laser.so">
+            <gaussianNoise>0.005</gaussianNoise>
+            <alwaysOn>true</alwaysOn>
+            <updateRate>${update_rate}</updateRate>
+            <topicName>${ros_topic}</topicName>
+            <frameName>/${name}_link</frameName>
+         </plugin>
+      </sensor>
     </gazebo>
   </xacro:macro>

File: youbot_common/youbot_description/urdf/youbot_base/base.gazebo.xacro (robot description, xacro)
@@ -38,5 +38,5 @@
 	<!-- position controller -->
 		<gazebo>
-      			<controller:gazebo_ros_p3d name="p3d_base_controller" plugin="libgazebo_ros_p3d.so">
+      			<plugin name="p3d_base_controller" filename="libgazebo_ros_p3d.so">
         			<alwaysOn>true</alwaysOn>
         			<updateRate>100.0</updateRate>
@@ -47,6 +47,5 @@
         			<xyzOffsets>25.7 25.7 0</xyzOffsets> <!-- initialize odometry for fake localization-->
         			<rpyOffsets>0 0 0</rpyOffsets>
-        			<interface:position name="p3d_base_position"/>
-      			</controller:gazebo_ros_p3d>
+      			</plugin>
       			<canonicalBody>base_footprint</canonicalBody>
     		</gazebo>
